File: hardware/eh_shield_04/wat.sch (KiCad schematic (older format))
At the start: 48 parts, among them P1 PINZA_1, P102 CAUDAL_2, P103 V_IN, P106 18b20, P109 LCD_I2C, P2 PINZA_5, P3 PINZA_2, P4 PINZA_6, P5 PINZA_3, P6 PINZA_4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

Commit message: cambios hacia PCB con presion
Connections:
- net labels added: intensidad_5, scl_pre_2, sda_int_6
- net labels removed: presion_2, scl_int_6, sda_int_5
Other:
- moved on the sheet: C10, C11, D1, P8, P9, R10
