File: hardware/eh_shield_04/wat.sch (KiCad schematic (older format))
At the start: 48 parts, among them P1 PINZA_1, P102 CAUDAL_2, P103 V_IN, P106 18b20, P109 LCD_I2C, P2 PINZA_5, P3 PINZA_2, P4 PINZA_6, P5 PINZA_3, P6 PINZA_4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

Commit message: hw wemos incluido
Parts:
- removed C106: 22uF, Capacitors_THT:CP_Radial_D5.0mm_P2.00mm, symbol CP1
- removed C3: 100nF, Capacitors_THT:C_Disc_D5.0mm_W2.5mm_P5.00mm, symbol C_Small
- removed R105, R106: 10K, oscar_libreria_huellas:Resistor_Horizontal_RM10mm, symbol R
- removed U101: ESP-12, oscar_libreria_huellas:ESP-07v2_pad, symbol ESP-12
- removed U104: LM1117, oscar_libreria_huellas:TO-220-LM117, symbol 7805
- removed W102: +3,3V, Wire_Pads:SolderWirePad_single_0-8mmDrill, symbol TEST_1P
- added U1: WeMos_mini, libreria_huellas_proyecto:D1_mini_board_direct, symbol WeMos_mini
Connections:
- net labels added: intensidad_5, presion_1, scl_int_6, sda_pre_2
- net labels removed: Ves_3V3, e_adc, e_cpd, e_g00, e_g02, e_g04, e_g05, e_g12, e_g13, e_g14, e_g15, e_g16, intensidad_6, presion_2, scl_pre_1, sda_int_5
- wire segments 143 -> 122
- no-connect marks 22 -> 24
