File: hardware/eh_shield_04/wat.kicad_pcb (KiCad board)
At the start: 2 copper layers, 101.8 x 85.9 mm, 44 parts, among them P1 PINZA_1, P102 CAUDAL_1, P103 V_IN, P106 18b20, P109 LCD_I2C, P110 ARD_DI_06, P111 ARD_ALI_04, P2 PINZA_7, P3 PINZA_2, P4 PINZA_8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

Commit message: cambios hacia PCB con presion
Parts:
- removed D104, D105: 1N4007, Diodes_ThroughHole:Diode_DO-35_SOD27_Horizontal_RM10
- removed P110: ARD_DI_06, Pin_Headers:Pin_Header_Straight_1x06
- removed P111: ARD_ALI_04, Pin_Headers:Pin_Header_Straight_1x04
- removed W103: +8V, Wire_Pads:SolderWirePad_single_0-8mmDrill
- added C10: 100nF, Capacitors_THT:C_Disc_D5.0mm_W2.5mm_P5.00mm, F.Cu at (123.4, 146.7)
- added C11: 100nF, Capacitors_THT:C_Disc_D5.0mm_W2.5mm_P5.00mm, F.Cu at (172.3, 91.2)
- added D1: 1N4007, oscar_libreria_huellas:Diode_DO-35_SOD27_Horizontal_RM10, F.Cu at (185.4, 66.0)
- added D2: 1N4148, Diodes_THT:D_A-405_P7.62mm_Horizontal, F.Cu at (159.1, 165.4)
- added D3: 1N4148, Diodes_THT:D_A-405_P7.62mm_Horizontal, F.Cu at (202.7, 139.4)
- added P7: MANO_2, oscar_libreria_huellas:bornier3, F.Cu at (123.3, 49.3)
- added P8: CAUDAL_1, oscar_libreria_huellas:bornier2, F.Cu at (173.0, 123.6)
- added R10: 10K, oscar_libreria_huellas:Resistor_Horizontal_RM10mm, F.Cu at (136.1, 168.4)
- added U106: NANO, oscar_libreria_huellas:arduino_nano, F.Cu at (111.1, 87.6)
- C9: value 220uF -> 100nF; footprint Capacitors_THT:CP_Radial_D5.0mm_P2.00mm -> Capacitors_THT:C_Disc_D5.0mm_W2.5mm_P5.00mm
- P102: value CAUDAL_1 -> CAUDAL_2
- P2: value PINZA_7 -> PINZA_5
- P4: value PINZA_8 -> PINZA_6
- P9: value INTENSIDAD -> MANO_1; footprint Pin_Headers:Pin_Header_Straight_1x08 -> oscar_libreria_huellas:bornier3
- R7: footprint Resistors_ThroughHole:Resistor_Horizontal_RM10mm -> oscar_libreria_huellas:Resistor_Horizontal_RM10mm
- moved P102 75.6 mm to (183.0, 123.6), turned to 0 degrees
- moved C9 74.3 mm to (112.0, 149.2)
- moved P9 71.1 mm to (155.4, 49.5), turned to 180 degrees
- moved C8 60.7 mm to (180.7, 115.4), turned to 0 degrees
- moved W101 51.6 mm to (201.9, 117.5)
- moved W102 41.8 mm to (62.4, 71.9)
- moved R106 26.4 mm to (78.0, 56.5)
- moved C106 15.2 mm to (98.3, 72.6), turned to 270 degrees
- moved U101 15.0 mm to (95.8, 52.7)
- moved P106 14.9 mm to (170.4, 49.5)
- moved U104 13.7 mm to (111.0, 73.0), turned to 180 degrees
- moved C3 12.5 mm to (92.5, 70.9), turned to 270 degrees
- moved R105 3.99 mm to (132.1, 68.7)
Connections:
- net /caudal_1 renamed /caudal_2
- C105 pad 1: /Vmp_12V -> /Vpc_5V
- C2 pad 2: /intensidad_7 -> /sda_int_5
- C5 pad 2: /intensidad_8 -> /intensidad_6
- C9 pad 1: /Var_8V -> /presion_2
- P109 pad 1: /sda -> /sda_int_5
- P109 pad 2: /scl -> /scl_pre_1
- P2 pad 1: /intensidad_7 -> /sda_int_5
- P4 pad 1: /intensidad_8 -> /intensidad_6
- P9 pad 1: /intensidad_1 -> /Vpc_5V
- P9 pad 2: /intensidad_2 -> /scl_pre_1
- P9 pad 3: /intensidad_3 -> GND
- R5 pad 2: /intensidad_7 -> /sda_int_5
- R7 pad 2: /intensidad_8 -> /intensidad_6
- U104 pad VI: /Var_8V -> /Vpc_5V
- W101 pad 1: /Vmp_12V -> /Vpc_5V
Routing:
- net /Var_8V: track 183.2 -> 0.00 mm
- net /Vpc_5V: track 110.2 -> 17.1 mm, vias 2 -> 0
- net /caudal_2: track 78.2 -> 0.26 mm
- net /intensidad_8: track 77.3 -> 0.00 mm
- net /intensidad_7: track 70.4 -> 0.00 mm
- net /18b20: track 57.7 -> 0.00 mm
- net /Ves_3V3: track 53.0 -> 0.00 mm
- net /sda: track 42.9 -> 0.00 mm
- net /e_tx: track 38.3 -> 0.00 mm
- net /scl: track 38.0 -> 0.00 mm
- net /e_rx: track 33.7 -> 0.00 mm
- net /e_rst: track 32.2 -> 0.00 mm
- net /sda_int_5: track 0.00 -> 24.7 mm
- net /intensidad_6: track 0.00 -> 24.4 mm
- net /Vmp_12V: track 24.2 -> 0.00 mm
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
Commit message: hw wemos incluido
Parts:
- removed C106: 22uF, Capacitors_ThroughHole:C_Radial_D5_L11_P2
- removed C3: 100nF, Capacitors_THT:C_Disc_D5.0mm_W2.5mm_P5.00mm
- removed R105, R106: 10K, Resistors_ThroughHole:Resistor_Horizontal_RM10mm
- removed U101: ESP-12, oscar_libreria_huellas:ESP-07v2_pad
- removed U104: LM1117, oscar_libreria_huellas:TO-220-LM117
- removed W102: +3,3V, Wire_Pads:SolderWirePad_single_0-8mmDrill
- added U1: WeMos_mini, libreria_huellas_proyecto:D1_mini_board_direct, F.Cu at (58.3, 44.8)
- moved C9 92.3 mm to (123.4, 57.7)
- moved R10 77.7 mm to (175.6, 101.5), turned to 270 degrees
- moved D2 73.7 mm to (186.3, 96.9), turned to 90 degrees
- moved C10 56.5 mm to (171.8, 117.5)
- moved W101 50.5 mm to (187.8, 69.0)
- moved D3 50.5 mm to (175.8, 96.8), turned to 90 degrees
- moved C11 38.1 mm to (155.6, 57.0)
- moved R2 35.0 mm to (186.6, 101.3), turned to 270 degrees
- moved U106 32.9 mm to (141.7, 75.6)
- moved R9 19.3 mm to (170.4, 56.5), turned to 270 degrees
- moved P109 15.4 mm to (144.7, 93.3), turned to 270 degrees
- moved R1 7.88 mm to (145.2, 99.9), turned to 180 degrees
- moved C8 2.47 mm to (182.1, 117.5)
Connections:
- net /Vpc_5V renamed VCC
- C11 pad 1: /scl_pre_1 -> /presion_1
- C2 pad 2: /sda_int_5 -> /intensidad_5
- C5 pad 2: /intensidad_6 -> /scl_int_6
- C9 pad 1: /presion_2 -> /sda_pre_2
- P109 pad 1: /sda_int_5 -> /scl_int_6
- P109 pad 2: /scl_pre_1 -> /sda_pre_2
- P2 pad 1: /sda_int_5 -> /intensidad_5
- P4 pad 1: /intensidad_6 -> /scl_int_6
- P7 pad 2: /presion_2 -> /sda_pre_2
- P9 pad 2: /scl_pre_1 -> /presion_1
- R5 pad 2: /sda_int_5 -> /intensidad_5
- R7 pad 2: /intensidad_6 -> /scl_int_6
- U106 pad 23: /sda_int_5 -> /sda_pre_2
- U106 pad 24: /scl_pre_1 -> /scl_int_6
- U106 pad 25: /intensidad_6 -> /intensidad_5
- U106 pad 26: /presion_2 -> /presion_1
Routing:
- net /sda_int_5: track 24.7 -> 0.00 mm
- net /intensidad_5: track 0.00 -> 24.7 mm
- net /scl_int_6: track 0.00 -> 24.4 mm
- net /intensidad_6: track 24.4 -> 0.00 mm
- net /intensidad_3: track 41.2 -> 24.0 mm
- net /intensidad_4: track 63.8 -> 49.9 mm
- net /intensidad_2: track 32.8 -> 21.7 mm
- net /intensidad_1: track 34.0 -> 24.3 mm
- net /Ref_medida: track 220.8 -> 215.7 mm
